File: nano_photogate.sch (KiCad schematic (older format))
At the start: 16 parts, among them P1 CONN_5X2, P2 CONN_4X2, P3 CONN_2X2, P4 CONN_4X2, P5 CONN_4X2, P6 CONN_4, P7 CONN_6X2, P8 CONN_6X2, P9 CONN_2, U1 ARDUINO_NANO

Commit message: Added problems/issues text to schematic.
Other:
- note added: "Problems/Issues:\n1. SPI header incorrect in layout - should be 5x2\n2. 3V3 is not connected on Arduino\n3. make I2C pullups selectable between 5V and 3V3"
Changed lines of the file:
@@
-EESchema Schematic File Version 2  date Mon 01 Aug 2011 07:15:24 PM PDT
+EESchema Schematic File Version 2  date Tue 27 Sep 2011 02:36:48 PM PDT
 LIBS:power
 LIBS:arduino_nano
@@
 LIBS:valves
 LIBS:nano_photogate-cache
-EELAYER 24  0
+EELAYER 25  0
 EELAYER END
 $Descr A4 11700 8267
@@
 Sheet 1 1
 Title ""
-Date "2 aug 2011"
+Date "27 sep 2011"
 Rev ""
 Comp ""
@@
 Comment4 ""
 $EndDescr
+Text Notes 1150 6700 0    60   ~ 0
+Problems/Issues:\n1. SPI header incorrect in layout - should be 5x2\n2. 3V3 is not connected on Arduino\n3. make I2C pullups selectable between 5V and 3V3
 NoConn ~ 2950 5300
 NoConn ~ 3700 2300
